Commit message: Cleaned up files. Added joint and state publishers.

File: src/pacman_config/model.urdf (robot description, URDF)
Before this commit: robot pacman, 16 links, 15 joints
Joints:
- joint GPS_Receiver_joint: origin xyz=0.0025924256a -0.170120818 0.759278136 rpy=0 0 0 -> xyz=0.0025924256 -0.170120818 0.759278136 rpy=0 0 0
- joint piksi_imu: origin xyz=0.0025924256a 0.170120818 0.759278136 rpy=0 0 0 -> xyz=-.0028890976 .1192403 .7526036923 rpy=0 0 0

Commit message: Runscripts, launch file and config changes.

File: src/pacman_config/model.urdf (robot description, URDF)
Before this commit: robot pacman, 16 links, 15 joints
Links:
- removed link Front_Camera
- removed link GPS_Receiver
- removed link os1/os1_imu
- added link os1/os1_sensor
- added link piksi_antenna
- added link webcam
Joints:
- removed joint Front_Camera_joint
- removed joint GPS_Receiver_joint
- removed joint os1/os1_imu_joint
- added joint os1/os1_sensor_joint: type fixed, parent base_link, child os1/os1_sensor, origin xyz=0 0 0.905932656 rpy=0 3.14159265359 -1.57079632679
- added joint piksi_antenna_joint: type fixed, parent base_link, child piksi_antenna, origin xyz=0.0025924256 -0.170120818 0.759278136 rpy=0 0 0
- added joint webcam_joint: type fixed, parent base_link, child webcam, origin xyz=0.152597358 0 0.77890116 rpy=0 0 0
- joint base_to_footprint_joint: child base_link -> base_footprint; parent base_footprint -> base_link
- joint piksi_imu: origin xyz=-.0028890976 .1192403 .7526036923 rpy=0 0 0 -> xyz=-.0028890976 .1192403 .7526036923 rpy=3.14159265359 0 0

Commit message: Decently working odometry with excellent point following.

File: src/pacman_config/model.urdf (robot description, URDF)
Before this commit: robot pacman, 16 links, 15 joints
Joints:
- joint os1/os1_sensor_joint: origin xyz=0 0 0.905932656 rpy=0 3.14159265359 -1.57079632679 -> xyz=0 0 0.905932656 rpy=3.14159265359 3.14159265359 -1.57079632679
